Commit message: last updated

File: src/pf_description/urdf/r2000.urdf.xacro (robot description, xacro)
@@ -4,5 +4,5 @@
         <link name="${prefix}scanner_link" >
             <visual>
-                <origin xyz="0 0 0" rpy="1.57 0 1.57" />
+                <origin xyz="0 0 0" rpy="0 0 0" />
                 <geometry>
                     <mesh filename="package://pf_description/meshes/R2000.stl" scale="0.001 0.001 0.001" />
@@ -10,7 +10,7 @@
             </visual>
             <collision>
-                <origin xyz="0 0 0.045" rpy="0 0 0" />
+                <origin xyz="-0.0058 0 -0.03885" rpy="0 0 0" />
                 <geometry>
-                    <box size="0.108 0.118 0.128" />
+                    <box size="0.118 0.108 0.117" />
                 </geometry>
             </collision>

File: src/pf_description/urdf/r2000_world.urdf.xacro (robot description, xacro)
@@ -1,4 +1,4 @@
 <?xml version="1.0"?>
-<robot xmlns:xacro="http://wiki.ros.org/xacro" name="r2300" >
+<robot xmlns:xacro="http://wiki.ros.org/xacro" name="r2000" >
     <xacro:include filename="$(find pf_description)/urdf/r2000.urdf.xacro" />
     <!-- create a virtual root link -->

File: src/pf_description/urdf/r2300.urdf.xacro (robot description, xacro)
@@ -4,5 +4,5 @@
         <link name="${prefix}scanner_link" >
             <visual>
-                <origin xyz="-0.00195 0.0158 -0.0094" rpy="-1.57 0 1.57" />
+                <origin xyz="0 0 0" rpy="0 0 0" />
                 <geometry>
                     <mesh filename="package://pf_description/meshes/R2300.stl" scale="0.001 0.001 0.001" />
@@ -10,7 +10,7 @@
             </visual>
             <collision>
-                <origin xyz="-0.00195 0.0158 -0.0094" rpy="-1.57 0 1.57" />
+                <origin xyz="0.01195 0.0158 -0.017" rpy="0 0 0" />
                 <geometry>
-                    <box size="0.0951 0.0685 0.0695" />
+                    <box size="0.07 0.0959 0.0586" />
                 </geometry>
             </collision>
